File: RaspiZeroCanDoCan.kicad_pcb (KiCad board)
At the start: 2 copper layers, 65 x 30 mm, 22 parts, among them IC1 MCP2562, P6 CAN_conn, P9 CAN_conn, U1 LD1117S50TR, U3 MCP2515-E/ST

Commit message: Update to Kicad5
Connections:
- Raspi1 pad 10: Net-(Raspi1-Pad10) -> (no net)
- Raspi1 pad 11: Net-(Raspi1-Pad11) -> (no net)
- Raspi1 pad 12: Net-(Raspi1-Pad12) -> (no net)
- Raspi1 pad 13: Net-(Raspi1-Pad13) -> (no net)
- Raspi1 pad 15: Net-(Raspi1-Pad15) -> (no net)
- Raspi1 pad 16: Net-(Raspi1-Pad16) -> (no net)
- Raspi1 pad 18: Net-(Raspi1-Pad18) -> (no net)
- Raspi1 pad 26: Net-(Raspi1-Pad26) -> (no net)
- Raspi1 pad 27: Net-(Raspi1-Pad27) -> (no net)
- Raspi1 pad 28: Net-(Raspi1-Pad28) -> (no net)
- Raspi1 pad 29: Net-(Raspi1-Pad29) -> (no net)
- Raspi1 pad 3: Net-(Raspi1-Pad3) -> (no net)
- Raspi1 pad 31: Net-(Raspi1-Pad31) -> (no net)
- Raspi1 pad 32: Net-(Raspi1-Pad32) -> (no net)
- Raspi1 pad 33: Net-(Raspi1-Pad33) -> (no net)
- Raspi1 pad 35: Net-(Raspi1-Pad35) -> (no net)
- Raspi1 pad 36: Net-(Raspi1-Pad36) -> (no net)
- Raspi1 pad 37: Net-(Raspi1-Pad37) -> (no net)
- Raspi1 pad 38: Net-(Raspi1-Pad38) -> (no net)
- Raspi1 pad 40: Net-(Raspi1-Pad40) -> (no net)
- Raspi1 pad 5: Net-(Raspi1-Pad5) -> (no net)
- Raspi1 pad 7: Net-(Raspi1-Pad7) -> (no net)
- Raspi1 pad 8: Net-(Raspi1-Pad8) -> (no net)
- U3 pad 11: Net-(U3-Pad11) -> (no net)
- U3 pad 12: Net-(U3-Pad12) -> (no net)
- U3 pad 15: Net-(U3-Pad15) -> (no net)
- U3 pad 3: Net-(U3-Pad3) -> (no net)
- U3 pad 4: Net-(U3-Pad4) -> (no net)
- U3 pad 5: Net-(U3-Pad5) -> (no net)
- U3 pad 6: Net-(U3-Pad6) -> (no net)
- U3 pad 7: Net-(U3-Pad7) -> (no net)
